File: pcb/version1.kicad_pcb (KiCad board)
At the start: 2 copper layers, 48 x 61.5 mm, 41 parts, among them J1 Conn_01x04_Female, J2 USB_B_Mini, J3 VO2_SPRING_PINS, U1 ACS711, U2 DRV78871, U3 ACS711, U4 STM32G030K6T6, U5 FT230XS, U6 MC33269

Commit message: updated hardware
Parts:
- removed BTN, RESET: SW_Push, Button_Switch_THT:SW_PUSH_6mm
- removed the J1 at (144.0, 54.0)
- removed R12: 500, Resistor_SMD:R_0603_1608Metric_Pad1.05x0.95mm_HandSolder
- added C10: 1uF, Capacitor_SMD:C_0603_1608Metric, F.Cu at (120.1, 69.7)
- added C11: 12pF, Capacitor_SMD:C_0603_1608Metric, F.Cu at (124.4, 63.8)
- added C12: 0.1uF, Capacitor_SMD:C_0603_1608Metric, F.Cu at (127.8, 85.6)
- added C13: 0.1uF, Capacitor_SMD:C_0603_1608Metric, F.Cu at (127.0, 69.8)
- added C14: 10nF, Capacitor_SMD:C_0603_1608Metric, F.Cu at (120.1, 68.1)
- added C15: 0.1uF, Capacitor_SMD:C_0603_1608Metric, F.Cu at (132.8, 100.0)
- added C16: 10uF, Capacitor_SMD:C_0603_1608Metric, F.Cu at (127.5, 97.2)
- added C18: 0.1uF, Capacitor_SMD:C_0603_1608Metric, F.Cu at (139.0, 57.2)
- added C19: 33pF, Capacitor_SMD:C_0603_1608Metric, F.Cu at (135.8, 97.2)
- added C20: 33pF, Capacitor_SMD:C_0603_1608Metric, F.Cu at (110.5, 65.5)
- added C21: 0.1uF, Capacitor_SMD:C_0603_1608Metric, F.Cu at (107.5, 68.2)
- added C22: 10uF, Capacitor_SMD:C_0603_1608Metric, F.Cu at (102.2, 65.5)
- added C23: 4.7uF, Capacitor_SMD:C_0603_1608Metric, F.Cu at (125.8, 97.2)
- added C24: 4.7uF, Capacitor_SMD:C_0603_1608Metric, F.Cu at (103.8, 68.2)
- added C9: 0.1uF, Capacitor_SMD:C_0603_1608Metric, F.Cu at (115.6, 74.5)
- added D10: ZMM5V6, Diode_SMD:D_MiniMELF, F.Cu at (107.6, 62.2)
- added D9: RED, LED_SMD:LED_0805_2012Metric, F.Cu at (123.4, 109.0)
- added H1: MountingHole_Pad, MountingHole:MountingHole_2.2mm_M2_Pad_Via, F.Cu at (144.5, 108.0)
- added H2: MountingHole_Pad, MountingHole:MountingHole_2.2mm_M2_Pad_Via, F.Cu at (103.5, 108.0)
- added H3: MountingHole_Pad, MountingHole:MountingHole_2.2mm_M2_Pad_Via, F.Cu at (103.5, 53.5)
- added H4: MountingHole_Pad, MountingHole:MountingHole_2.2mm_M2_Pad_Via, F.Cu at (144.5, 53.5)
- added J3: Screw_Terminal_01x02, TerminalBlock_MetzConnect:TerminalBlock_MetzConnect_Type055_RT01502HDWU_1x02_P5.00mm_Horizontal, F.Cu at (130.0, 107.0)
- added J4: Conn_01x04_Female, Connector_PinSocket_2.54mm:PinSocket_1x04_P2.54mm_Vertical, F.Cu at (144.5, 59.4)
- added L1: 39nH, Inductor_SMD:L_0402_1005Metric, F.Cu at (120.1, 66.8)
- added L2: 2.2uH, Inductor_SMD:L_0805_2012Metric, F.Cu at (129.5, 97.2)
- added L3: 2.2uH, Inductor_SMD:L_0805_2012Metric, F.Cu at (104.2, 65.5)
- added Q1: AO3400A, Package_TO_SOT_SMD:SOT-23, F.Cu at (143.5, 95.0)
- added R13: 1k, Resistor_SMD:R_0603_1608Metric, F.Cu at (137.2, 57.2)
- added R16: 124k, Resistor_SMD:R_0603_1608Metric, F.Cu at (112.2, 65.5)
- added R17: 23.7k, Resistor_SMD:R_0603_1608Metric, F.Cu at (114.0, 65.5)
- added R18: 4.7k, Resistor_SMD:R_0603_1608Metric, F.Cu at (115.6, 77.8)
- added R19: 9.1k, Resistor_SMD:R_0603_1608Metric, F.Cu at (115.6, 76.2)
- added R2: 124k, Resistor_SMD:R_0603_1608Metric, F.Cu at (137.5, 97.2)
- added R20: 4.7k, Resistor_SMD:R_0603_1608Metric, F.Cu at (115.6, 71.1)
- added R21: 9.1k, Resistor_SMD:R_0603_1608Metric, F.Cu at (115.6, 72.8)
- added R22: 47, Resistor_SMD:R_0603_1608Metric, F.Cu at (122.5, 69.0)
- added SW1: SW_Push, Button_Switch_THT:SW_PUSH_6mm, F.Cu at (113.5, 55.0)
- added SW3: SW_Push, Button_Switch_THT:SW_PUSH_6mm, F.Cu at (128.0, 55.0)
- added U7: MP2451, Package_TO_SOT_SMD:SOT-23-6, F.Cu at (107.5, 65.5)
- added Y1: 16MHz, Crystal:Crystal_SMD_SeikoEpson_FA238-4Pin_3.2x2.5mm, F.Cu at (125.5, 67.3)
- C1, C2: value 0.1uF -> 2.2uF; footprint Capacitor_SMD:C_0603_1608Metric_Pad1.05x0.95mm_HandSolder -> Capacitor_SMD:C_0603_1608Metric
- C3: value 0.1uF -> 1nF; footprint Capacitor_SMD:C_0603_1608Metric_Pad1.05x0.95mm_HandSolder -> Capacitor_SMD:C_0603_1608Metric
- C4: value 4.7uF -> 1nF; footprint Capacitor_SMD:C_1206_3216Metric_Pad1.42x1.75mm_HandSolder -> Capacitor_SMD:C_0603_1608Metric
- C5: value 47pF -> 4.7uF; footprint Capacitor_SMD:C_0603_1608Metric_Pad1.05x0.95mm_HandSolder -> Capacitor_SMD:C_0603_1608Metric
- C6: value 47pF -> 0.1uF; footprint Capacitor_SMD:C_0603_1608Metric_Pad1.05x0.95mm_HandSolder -> Capacitor_SMD:C_0603_1608Metric
- C7: value 1uF -> 12pF; footprint Capacitor_SMD:C_0603_1608Metric_Pad1.05x0.95mm_HandSolder -> Capacitor_SMD:C_0603_1608Metric
- C8: value 10uF -> 0.1uF; footprint Capacitor_SMD:C_1206_3216Metric_Pad1.42x1.75mm_HandSolder -> Capacitor_SMD:C_0603_1608Metric
- D1, D2: value LED -> B5819W; footprint LED_SMD:LED_0603_1608Metric_Pad1.05x0.95mm_HandSolder -> Diode_SMD:D_SOD-123
- D3: value LED -> ZMM3V3; footprint LED_SMD:LED_0603_1608Metric_Pad1.05x0.95mm_HandSolder -> Diode_SMD:D_MiniMELF
- D4, D5, D6: value LED -> GREEN; footprint LED_SMD:LED_0603_1608Metric_Pad1.05x0.95mm_HandSolder -> LED_SMD:LED_0805_2012Metric
- D7, D8: value D_Schottky -> GREEN; footprint Diode_SMD:D_0603_1608Metric -> LED_SMD:LED_0805_2012Metric
- JP2: renamed from JP1; value SolderJumper_2_Open -> Solder Bridge
- JP3: renamed from JP2; value SolderJumper_2_Open -> Solder Bridge
- R1: value 100k -> 10k; footprint Resistor_SMD:R_0603_1608Metric_Pad1.05x0.95mm_HandSolder -> Resistor_SMD:R_0603_1608Metric
- R10, R11: value 500 -> 4.7k; footprint Resistor_SMD:R_0603_1608Metric_Pad1.05x0.95mm_HandSolder -> Resistor_SMD:R_0603_1608Metric
- R15: renamed from R2; footprint Resistor_SMD:R_0603_1608Metric_Pad1.05x0.95mm_HandSolder -> Resistor_SMD:R_0603_1608Metric
- R3: value 27 -> 40.2k; footprint Resistor_SMD:R_0603_1608Metric_Pad1.05x0.95mm_HandSolder -> Resistor_SMD:R_0603_1608Metric
- R4: value 5.1M -> 500; footprint Resistor_SMD:R_0603_1608Metric_Pad1.05x0.95mm_HandSolder -> Resistor_SMD:R_0603_1608Metric
- R5: value 1M -> 500; footprint Resistor_SMD:R_0603_1608Metric_Pad1.05x0.95mm_HandSolder -> Resistor_SMD:R_0603_1608Metric
- R6: value 27 -> 500; footprint Resistor_SMD:R_0603_1608Metric_Pad1.05x0.95mm_HandSolder -> Resistor_SMD:R_0603_1608Metric
- R7, R8, R9: footprint Resistor_SMD:R_0603_1608Metric_Pad1.05x0.95mm_HandSolder -> Resistor_SMD:R_0603_1608Metric
- U1, U3: value ACS711 -> ACS712xLCTR-05B
- U2: value DRV78871 -> STM32F405RGTx; footprint vo2_test_fixture:DRV7881 -> Package_QFP:LQFP-64_10x10mm_P0.5mm
- U4: value STM32G030K6T6 -> MP2451; footprint Package_QFP:LQFP-32_7x7mm_P0.8mm -> Package_TO_SOT_SMD:SOT-23-6
- U5: value FT230XS -> M24C02-WMN; footprint Package_SO:SSOP-16_3.9x4.9mm_P0.635mm -> Package_SO:SOIC-8_3.9x4.9mm_P1.27mm
- U6: value MC33269 -> USBLC6-2P6; footprint Package_SO:SOIC-8_3.9x4.9mm_P1.27mm -> Package_TO_SOT_SMD:SOT-666
- moved R15 40.8 mm to (140.8, 57.2), turned to 270 degrees
- moved R9 40.8 mm to (125.4, 109.0), turned to 90 degrees
- moved C7 39.8 mm to (126.6, 63.8)
- moved D6 39.1 mm to (140.2, 76.9), turned to 180 degrees
- moved D8 37.0 mm to (140.2, 81.9)
- moved D7 34.8 mm to (140.2, 79.4), turned to 180 degrees
- moved R4 32.8 mm to (144.0, 71.9), turned to 180 degrees
- moved D3 30.0 mm to (127.8, 100.4)
- moved C2 29.9 mm to (131.1, 85.6), turned to 270 degrees
- moved R5 29.8 mm to (144.0, 74.4), turned to 180 degrees
- moved U5 28.1 mm to (133.3, 65.0)
- moved C8 27.5 mm to (132.3, 73.6), turned to 0 degrees
- moved R6 27.3 mm to (144.0, 76.9), turned to 180 degrees
- moved U1 26.7 mm to (107.5, 78.5), turned to 0 degrees
- moved D2 26.3 mm to (122.2, 95.8)
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- renumbered J2 to J1, J3 to J2
Connections:
- net /HEAT_OUT1 renamed /HEAT_PULSE_1
- net /HEAT_OUT2 renamed /HEAT_PULSE_2
- C1 pad 1: /RST -> Net-(C1-Pad1)
- C2 pad 1: /BTN -> Net-(C2-Pad1)
- C3 pad 1: +3V3 -> Net-(C3-Pad1)
- C4 pad 1: +3V3 -> Net-(C4-Pad1)
- C5 pad 1: Net-(C5-Pad1) -> +3V3
- C6 pad 1: Net-(C6-Pad1) -> +3V3
- C7 pad 1: /POWER_SRC -> /OSC_IN
- D1 pad 1: Net-(D1-Pad1) -> /VPOWER
- D1 pad 2: /LED1 -> VBUS
- D2 pad 1: Net-(D2-Pad1) -> /VPOWER
- D2 pad 2: /LED2 -> +15V
- D3 pad 1: Net-(D3-Pad1) -> Net-(C15-Pad2)
- D3 pad 2: /LED3 -> GND
- D4 pad 2: /LED4 -> /LED1
- D5 pad 2: /LED5 -> /LED2
- D6 pad 2: +3V3 -> /LED3
- D7 pad 1: /POWER_SRC -> Net-(D7-Pad1)
- D7 pad 2: Net-(D7-Pad2) -> /LED4
- D8 pad 1: /POWER_SRC -> Net-(D8-Pad1)
- D8 pad 2: +15V -> /LED5
- J1 pad 1: Net-(D7-Pad2) -> VBUS
- J1 pad 2: Net-(C6-Pad1) -> /USB_CONN_D-
- J1 pad 3: Net-(C5-Pad1) -> /USB_CONN_D+
- J1 pad 6: GND -> Net-(J1-Pad6)
- J2 pad 3: /HEAT_LOW -> /HEAT_GND
- J2 pad 4: /HEAT_LOW -> /HEAT_GND
- R1 pad 2: /RST -> Net-(R1-Pad2)
- R10 pad 1: Net-(D4-Pad1) -> +3V3
- R10 pad 2: GND -> /I2C_SDA
- R11 pad 1: Net-(D5-Pad1) -> /I2C_SCL
- R11 pad 2: GND -> +3V3
- R3 pad 1: Net-(R3-Pad1) -> GND
- R3 pad 2: Net-(C5-Pad1) -> Net-(C19-Pad2)
- R4 pad 1: +15V -> GND
- R4 pad 2: /ADC_16V -> Net-(D4-Pad1)
- R5 pad 1: /ADC_16V -> GND
- R5 pad 2: GND -> Net-(D5-Pad1)
- R6 pad 1: Net-(R6-Pad1) -> GND
- R6 pad 2: Net-(C6-Pad1) -> Net-(D6-Pad1)
- R7 pad 1: Net-(D1-Pad1) -> GND
- R7 pad 2: GND -> Net-(D7-Pad1)
- R8 pad 1: Net-(D2-Pad1) -> GND
- R8 pad 2: GND -> Net-(D8-Pad1)
- R9 pad 1: Net-(D3-Pad1) -> GND
- R9 pad 2: GND -> Net-(D9-Pad1)
- U1 pad 1: /HEAT_SENSE -> +15V
- U1 pad 2: /HEAT_SENSE -> +15V
- U1 pad 6: Net-(U1-Pad6) -> Net-(C3-Pad1)
- U1 pad 7: /ADC_HEAT1 -> /CURRENT1
- U1 pad 8: +3V3 -> +5V
- U2 pad 1: /PWM_HEAT -> +3V3
- U2 pad 2: GND -> Net-(U2-Pad2)
- U2 pad 3: +15V -> Net-(U2-Pad3)
- U2 pad 4: GND -> Net-(U2-Pad4)
- U2 pad 5: /HEAT_LOW -> /OSC_IN
- U2 pad 6: /HEAT_SENSE -> /OSC_OUT
- U3 pad 1: /HEAT_SENSE -> +15V
- U3 pad 2: /HEAT_SENSE -> +15V
- U3 pad 6: Net-(U3-Pad6) -> Net-(C4-Pad1)
- U3 pad 7: /ADC_HEAT2 -> /CURRENT2
- U3 pad 8: +3V3 -> +5V
- U4 pad 2: Net-(U4-Pad2) -> GND
- U4 pad 3: Net-(U4-Pad3) -> Net-(C19-Pad2)
- U4 pad 5: GND -> /VPOWER
- U4 pad 6: /RST -> Net-(C15-Pad2)
- U5 pad 1: /UART_RX -> GND
- U5 pad 2: /UART_CTS -> GND
- U5 pad 3: +3V3 -> GND
- U5 pad 4: /UART_TX -> GND
- U5 pad 5: GND -> /I2C_SDA
- U5 pad 6: /UART_RTS -> /I2C_SCL
- U5 pad 7: Net-(U5-Pad7) -> GND
- U5 pad 8: Net-(R3-Pad1) -> +3V3
- U6 pad 1: GND -> /USB_CONN_D-
- U6 pad 2: +3V3 -> GND
- U6 pad 3: +3V3 -> /USB_CONN_D+
- U6 pad 4: /POWER_SRC -> /USB_D+
- U6 pad 5: Net-(U6-Pad5) -> VBUS
- U6 pad 6: +3V3 -> /USB_D-
Routing:
- net /RST: track 43.5 -> 0.00 mm, vias 2 -> 0
- net /HEAT_PULSE_1: track 47.4 -> 6.56 mm
- net Net-(R1-Pad2): track 0.00 -> 33.4 mm, vias 0 -> 1
- net +5V: track 0.00 -> 29.3 mm, vias 0 -> 2
- net /ADC_HEAT1: track 24.0 -> 0.00 mm, vias 2 -> 0
- net /HEAT_PULSE_2: track 42.6 -> 19.2 mm
- net +3V3: track 128.0 -> 149.6 mm, vias 8 -> 6
- net /VPOWER: track 0.00 -> 20.8 mm, vias 0 -> 2
- net /USB_D-: track 0.00 -> 20.6 mm
- net /USB_D+: track 0.00 -> 20.0 mm
- net /ADC_16V: track 19.6 -> 0.00 mm, vias 2 -> 0
- net /ADC_HEAT2: track 17.8 -> 0.00 mm, vias 2 -> 0
- net VBUS: track 0.00 -> 17.5 mm
- net GND: track 36.6 -> 53.2 mm, vias 30 -> 42
- net Net-(C21-Pad2): track 0.00 -> 16.3 mm, vias 0 -> 2
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- added copper zone on F.Cu, net /HEAT_PULSE_1
- added copper zone on F.Cu, net /HEAT_PULSE_2
- added copper zone on F.Cu, net Net-(J1-Pad6)
- removed copper zone on F.Cu, net +3V3
- removed copper zone on B.Cu, net /HEAT_LOW
- removed copper zone on F.Cu, net /HEAT_SENSE
- removed copper zone on F.Cu, net Net-(J2-Pad1)
- removed copper zone on F.Cu, net Net-(J2-Pad2)
Other:
- rule via_min_size: 0.4 -> 0.45
- board text added: "+"
- board text added: "-"
- board text added: "JLCJLCJLCJLC"
- board text added: "RESET"
- board text added: "START"
