File: pcb/version1.sch (KiCad schematic (older format))
At the start: 53 parts, among them J1 AlligatorClip, J10 Conn_01x01_Male, J11 AlligatorClip, J12 AlligatorClip, J2 AlligatorClip, J3 Conn_01x02_Female, J4 Conn_01x04_Female, J5 USB_B_Mini, J6 Conn_01x04_Female, J7 Conn_01x01_Male, J8 Conn_01x01_Male, J9 Conn_01x01_Male, SW1 SW_Push, SW2 SW_Push, U1 ACS711, U2 ACS711, U3 STM32G030K6T6, U4 FT230XS, U5 MC33269, Y1 12MHz

Commit message: updated hardware design
Parts:
- removed C3, C4: 18pF, Capacitor_SMD:C_0603_1608Metric_Pad1.05x0.95mm_HandSolder, symbol Device:C
- removed D6, D8: LED, LED_SMD:LED_0603_1608Metric_Pad1.05x0.95mm_HandSolder, symbol Device:LED
- removed J1, J11, J12, J2: AlligatorClip, vo2_test_fixture:AlligatorPowerPads, symbol vo2_test_fixture:AlligatorClip
- removed J10, J7, J8, J9: Conn_01x01_Male, Connector_PinHeader_2.00mm:PinHeader_1x01_P2.00mm_Vertical, symbol Connector:Conn_01x01_Male
- removed J3: Conn_01x02_Female, vo2_test_fixture:PinHeader_2x3.5mm, symbol Connector:Conn_01x02_Female
- removed J4: Conn_01x04_Female, Connector_PinSocket_2.54mm:PinSocket_1x04_P2.54mm_Vertical, symbol Connector:Conn_01x04_Female
- removed R13: 300, Resistor_SMD:R_0603_1608Metric_Pad1.05x0.95mm_HandSolder, symbol Device:R_US
- removed R15: 1.5k, Resistor_SMD:R_0603_1608Metric_Pad1.05x0.95mm_HandSolder, symbol Device:R_US
- removed R3: 1M, Resistor_SMD:R_0603_1608Metric_Pad1.05x0.95mm_HandSolder, symbol Device:R_US
- removed Y1: 12MHz, Crystal:Crystal_SMD_HC49-SD, symbol Device:Crystal
- added D7, D8: D_Schottky, Diode_SMD:D_0603_1608Metric, symbol Device:D_Schottky
- added J3: VO2_SPRING_PINS, vo2_test_fixture:SPRING_PINS, symbol vo2_test_fixture:VO2_SPRING_PINS
- added JP1, JP2: SolderJumper_2_Open, Jumper:SolderJumper-2_P1.3mm_Open_RoundedPad1.0x1.5mm, symbol Jumper:SolderJumper_2_Open
- added U2: DRV78871, vo2_test_fixture:DRV7881, symbol vo2_test_fixture:DRV78871
- R10: renamed from R11; value 300 -> 500
- R11: renamed from R12; value 300 -> 500
- R12: renamed from R14; value 300 -> 500
- R7: renamed from R8; value 300 -> 500
- R8: renamed from R9; value 300 -> 500
- R9: renamed from R10; value 300 -> 500
- renumbered C5 to C3, C6 to C4, C7 to C5, C8 to C6, C9 to C7, C10 to C8, D7 to D6, J6 to J1, J5 to J2, R4 to R3, R5 to R4, R6 to R5, R7 to R6, U2 to U3, U3 to U4, U4 to U5, U5 to U6
Connections:
- net labels added: HEAT_LOW, HEAT_SENSE, POWER_SRC
- net labels removed: HEAT_IN, OSC1, OSC2
- wire segments 230 -> 200
Other:
- note added: "Motor Controller"
- note removed: "Clock"
- note removed: "Motor Controller Inputs"
- note removed: "Motor Controller Outputs"
- note removed: "Power Connector"
- moved on the sheet: C5, C6, C7, C8, D1, D2, D3, D4, D5, D6, J1, R10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

Commit message: updated hardware
Parts:
- removed C1, C2, C3: 0.1uF, Capacitor_SMD:C_0603_1608Metric_Pad1.05x0.95mm_HandSolder, symbol Device:C
- removed C4: 4.7uF, Capacitor_SMD:C_1206_3216Metric_Pad1.42x1.75mm_HandSolder, symbol Device:CP1
- removed C5, C6: 47pF, Capacitor_SMD:C_0603_1608Metric_Pad1.05x0.95mm_HandSolder, symbol Device:C
- removed C7: 1uF, Capacitor_SMD:C_0603_1608Metric_Pad1.05x0.95mm_HandSolder, symbol Device:CP1
- removed C8: 10uF, Capacitor_SMD:C_1206_3216Metric_Pad1.42x1.75mm_HandSolder, symbol Device:CP1
- removed D1, D2, D3, D4, D5, D6: LED, LED_SMD:LED_0603_1608Metric_Pad1.05x0.95mm_HandSolder, symbol Device:LED
- removed D7, D8: D_Schottky, Diode_SMD:D_0603_1608Metric, symbol Device:D_Schottky
- removed R1: 100k, Resistor_SMD:R_0603_1608Metric_Pad1.05x0.95mm_HandSolder, symbol Device:R_US
- removed R10, R11, R12, R7, R8, R9: 500, Resistor_SMD:R_0603_1608Metric_Pad1.05x0.95mm_HandSolder, symbol Device:R_US
- removed R3, R6: 27, Resistor_SMD:R_0603_1608Metric_Pad1.05x0.95mm_HandSolder, symbol Device:R_US
- removed R4: 5.1M, Resistor_SMD:R_0603_1608Metric_Pad1.05x0.95mm_HandSolder, symbol Device:R_US
- removed R5: 1M, Resistor_SMD:R_0603_1608Metric_Pad1.05x0.95mm_HandSolder, symbol Device:R_US
- removed SW2: SW_Push, Button_Switch_THT:SW_PUSH_6mm, symbol Switch:SW_Push
- removed U1, U3: ACS711, Package_SO:SOIC-8_3.9x4.9mm_P1.27mm, symbol vo2_test_fixture:ACS711
- removed U2: DRV78871, vo2_test_fixture:DRV7881, symbol vo2_test_fixture:DRV78871
- removed U4: STM32G030K6T6, Package_QFP:LQFP-32_7x7mm_P0.8mm, symbol vo2_test_fixture:STM32G030K6T6
- removed U5: FT230XS, Package_SO:SSOP-16_3.9x4.9mm_P0.635mm, symbol Interface_USB:FT230XS
- removed U6: MC33269, Package_SO:SOIC-8_3.9x4.9mm_P1.27mm, symbol vo2_test_fixture:MC33269
- added C1, C2: 2.2uF, Capacitor_SMD:C_0603_1608Metric, symbol Device:C_Small
- added C10: 1uF, Capacitor_SMD:C_0603_1608Metric, symbol Device:C_Small
- added C11, C7: 12pF, Capacitor_SMD:C_0603_1608Metric, symbol Device:C_Small
- added C12, C13, C15, C21, C6, C8, C9: 0.1uF, Capacitor_SMD:C_0603_1608Metric, symbol Device:C_Small
- added C14: 10nF, Capacitor_SMD:C_0603_1608Metric, symbol Device:C_Small
- added C16, C22: 10uF, Capacitor_SMD:C_0603_1608Metric, symbol Device:C_Small
- added C18: 0.1uF, Capacitor_SMD:C_0603_1608Metric, symbol Device:C
- added C19, C20: 33pF, Capacitor_SMD:C_0603_1608Metric, symbol Device:C_Small
- added C23, C24, C5: 4.7uF, Capacitor_SMD:C_0603_1608Metric, symbol Device:C_Small
- added C3, C4: 1nF, Capacitor_SMD:C_0603_1608Metric, symbol Device:C_Small
- added D1, D2: B5819W, Diode_SMD:D_SOD-123, symbol Device:D_Small_ALT
- added D10: ZMM5V6, Diode_SMD:D_MiniMELF, symbol Device:D_Zener_Small_ALT
- added D3: ZMM3V3, Diode_SMD:D_MiniMELF, symbol Device:D_Zener_Small_ALT
- added D4, D5, D6, D7, D8: GREEN, LED_SMD:LED_0805_2012Metric, symbol Device:LED_Small_ALT
- added D9: RED, LED_SMD:LED_0805_2012Metric, symbol Device:LED_Small_ALT
- added H1, H2, H3, H4: MountingHole_Pad, MountingHole:MountingHole_2.2mm_M2_Pad_Via, symbol Mechanical:MountingHole_Pad
- added J3: Screw_Terminal_01x02, TerminalBlock_MetzConnect:TerminalBlock_MetzConnect_Type055_RT01502HDWU_1x02_P5.00mm_Horizontal, symbol Connector:Screw_Terminal_01x02
- added L1: 39nH, Inductor_SMD:L_0402_1005Metric, symbol Device:L_Small
- added L2, L3: 2.2uH, Inductor_SMD:L_0805_2012Metric, symbol Device:L_Small
- added Q1: AO3400A, Package_TO_SOT_SMD:SOT-23, symbol Device:Q_NMOS_GSD
- added R1: 10k, Resistor_SMD:R_0603_1608Metric, symbol Device:R_Small_US
- added R10, R11, R18, R20: 4.7k, Resistor_SMD:R_0603_1608Metric, symbol Device:R_Small_US
- added R13: 1k, Resistor_SMD:R_0603_1608Metric, symbol Device:R_US
- added R16, R2: 124k, Resistor_SMD:R_0603_1608Metric, symbol Device:R_Small_US
- added R17: 23.7k, Resistor_SMD:R_0603_1608Metric, symbol Device:R_Small_US
- added R19, R21: 9.1k, Resistor_SMD:R_0603_1608Metric, symbol Device:R_Small_US
- added R22: 47, Resistor_SMD:R_0603_1608Metric, symbol Device:R_Small_US
- added R3: 40.2k, Resistor_SMD:R_0603_1608Metric, symbol Device:R_Small_US
- added R4, R5, R6, R7, R8, R9: 500, Resistor_SMD:R_0603_1608Metric, symbol Device:R_Small_US
- added SW3: SW_Push, Button_Switch_THT:SW_PUSH_6mm, symbol Switch:SW_Push
- added U1, U3: ACS712xLCTR-05B, Package_SO:SOIC-8_3.9x4.9mm_P1.27mm, symbol Sensor_Current:ACS712xLCTR-05B
- added U2: STM32F405RGTx, Package_QFP:LQFP-64_10x10mm_P0.5mm, symbol MCU_ST_STM32F4:STM32F405RGTx
- added U4, U7: MP2451, Package_TO_SOT_SMD:SOT-23-6, symbol vo2_test_fixture:MP2451
- added U5: M24C02-WMN, Package_SO:SOIC-8_3.9x4.9mm_P1.27mm, symbol Memory_EEPROM:M24C02-WMN
- added U6: USBLC6-2P6, Package_TO_SOT_SMD:SOT-666, symbol Power_Protection:USBLC6-2P6
- added Y1: 16MHz, Crystal:Crystal_SMD_SeikoEpson_FA238-4Pin_3.2x2.5mm, symbol Device:Crystal_GND24_Small
- JP2: renamed from JP1; value SolderJumper_2_Open -> Solder Bridge
- JP3: renamed from JP2; value SolderJumper_2_Open -> Solder Bridge
- R15: renamed from R2; footprint Resistor_SMD:R_0603_1608Metric_Pad1.05x0.95mm_HandSolder -> Resistor_SMD:R_0603_1608Metric
- renumbered J2 to J1, J3 to J2, J1 to J4
Connections:
- net +15V: now also C24.1, D2.2 (A), J3.2 (Pin_2), U1.1 (IP+), U1.2 (IP+), U3.1 (IP+), U3.2 (IP+), U7.5 (VIN)
- net +3V3: now also C12.1, C13.1, C16.1, C19.1, C5.1, C6.1, C8.1, C9.1, D9.2 (A), L1.1, L2.2, R1.1, R10.1, R11.2, R2.2, U2.1 (VBAT), U2.19 (VDD), U2.32 (VDD), U2.48 (VDD), U2.64 (VDD), U4.4 (EN), U5.8 (VCC)
- net BTN: now also C18.1, R13.1, U2.22 (PA6)
- net GND: now also C1.2, C10.2, C11.2, C12.2, C13.2, C14.2, C16.2, C18.2, C2.2, C22.2, C23.2, C24.2, C3.2, C4.2, C5.2, C6.2, C7.2, C8.2, C9.2, D10.2 (A), D3.2 (A), H1.1, H2.1, H3.1, H4.1, J3.1 (Pin_1), Q1.2 (S), R17.1, R19.1, R21.1, R3.1, R4.1, R5.1, R6.1, R7.1, R8.1, R9.1, SW3.1, U1.5 (GND), U2.12 (VSSA), U2.18 (VSS), U2.63 (VSS), U3.5 (GND), U4.2 (GND), U5.1 (E0), U5.2 (E1), U5.3 (E2), U5.4 (VSS), U5.7 (~WC), U6.2 (GND), U7.2 (GND), Y1.2, Y1.4; no longer J1.6 (Shield)
- net LED1: now also D4.2 (A), U2.56 (PB4)
- net LED2: now also D5.2 (A), U2.55 (PB3)
- net LED3: now also D6.2 (A), U2.54 (PD2)
- net LED4: now also D7.2 (A), U2.53 (PC12)
- net LED5: now also D8.2 (A), U2.52 (PC11)
- net PWM_HEAT: now also Q1.1 (G), U2.41 (PA8)
- net RST: now also U2.7 (NRST); no longer SW1.2
- net SWCLK: now also U2.49 (PA14)
- net SWDIO: now also U2.46 (PA13)
- net VBUS: now reaches J1.1 (VBUS)
- net VBUS: now also D1.2 (A), U6.5 (VBUS)
- net USB_CONN_D-: now reaches J1.2 (D-)
- net USB_CONN_D-: now also U6.1 (I/O1)
- net USB_CONN_D+: now reaches J1.3 (D+)
- net USB_CONN_D+: now also U6.3 (I/O2)
- net HEAT_LOW renamed HEAT_GND
- net HEAT_GND: now also Q1.3 (D)
- net HEAT_OUT1 renamed HEAT_PULSE_1
- net HEAT_PULSE_1: now also U1.3 (IP-), U1.4 (IP-)
- net HEAT_OUT2 renamed HEAT_PULSE_2
- net HEAT_PULSE_2: now also U3.3 (IP-), U3.4 (IP-)
- new net: R18.1, R19.2, U2.14 (PA0)
- new net: R20.1, R21.2, U2.15 (PA1)
- new net: C1.1, U2.31 (VCAP_1)
- new net: C2.1, U2.47 (VCAP_2)
- new net: R1.2, SW1.2, U2.60 (BOOT0)
- new net: C15.2, D3.1 (K), L2.1, U4.6 (SW)
- new net: C21.1, U7.1 (BST)
- new net: C20.2, R16.1, R17.2, U7.3 (FB)
- new net: C21.2, D10.1 (K), L3.1, U7.6 (SW)
- new net: C11.1, R22.1, Y1.3
- new net: R13.2, SW3.2
- new net: C19.2, R2.1, R3.2, U4.3 (FB)
- new net: C15.1, U4.1 (BST)
- new net: D4.1 (K), R4.2
- new net: D5.1 (K), R5.2
- new net: D6.1 (K), R6.2
- new net: D7.1 (K), R7.2
- new net: D8.1 (K), R8.2
- new net: D9.1 (K), R9.2
- new net: C3.1, U1.6 (FILTER)
- new net: C4.1, U3.6 (FILTER)
- new net +3.3VA: C10.1, C14.1, L1.2, U2.13 (VDDA)
- new net +5V: C20.1, C22.1, L3.2, R16.2, U1.8 (VCC), U3.8 (VCC), U7.4 (EN)
- new net CURRENT1: R18.2, U1.7 (VIOUT)
- new net CURRENT2: R20.2, U3.7 (VIOUT)
- new net I2C_SCL: R11.1, U2.58 (PB6), U5.6 (SCL)
- new net I2C_SDA: R10.2, U2.59 (PB7), U5.5 (SDA)
- new net OSC_IN: C7.1, U2.5 (PH0), Y1.1
- new net OSC_OUT: R22.2, U2.6 (PH1)
- new net USB_D+: U2.45 (PA12), U6.4 (I/O2)
- new net USB_D-: U2.44 (PA11), U6.6 (I/O1)
- new net VPOWER: C23.1, D1.1 (K), D2.1 (K), U4.5 (VIN)
- no-connect marks 2 -> 36
Other:
- note added: "5V Regulator"
- note added: "EEPROM"
- note added: "ESD Protection"
- note added: "Mounting holes"
- note added: "Oscillator"
- note added: "Power Terminal"
- note added: "Power supply filtering"
- note added: "USB Connector"
- note added: "Voltage Switching"
- note removed: "Motor Controller"
- note removed: "Reset button"
- note removed: "USB-UART Converter"
- moved on the sheet: J1, J4, R15
